Commit message: use stl files from submodule

File: urdf/claw.xacro (robot description, xacro)
@@ -12,5 +12,5 @@
     <visual>
       <geometry>
-        <mesh scale="0.001 0.001 0.001" filename="package://${package_name}/meshes/dragon_claw_palm.stl"/>
+        <mesh scale="0.001 0.001 0.001" filename="package://${package_name}/openscad/stl/dragon_claw_palm.stl"/>
       </geometry>
       <origin rpy="0 0 0" xyz="0 0 0"/>
@@ -29,5 +29,5 @@
       <visual>
         <geometry>
-          <mesh scale="0.001 0.001 0.001" filename="package://${package_name}/meshes/dragon_claw_knuckle_${digit}.stl"/>
+          <mesh scale="0.001 0.001 0.001" filename="package://${package_name}/openscad/stl/dragon_claw_knuckle_${digit}.stl"/>
         </geometry>
         <origin xyz="0 0 0" rpy="0 0 0"/>
@@ -47,5 +47,5 @@
       <visual>
         <geometry>
-          <mesh scale="0.001 0.001 0.001" filename="package://${package_name}/meshes/dragon_claw_finger_${digit}.stl"/>
+          <mesh scale="0.001 0.001 0.001" filename="package://${package_name}/openscad/stl/dragon_claw_finger_${digit}.stl"/>
         </geometry>
         <origin xyz="0 0 0" rpy="0 0 0"/>
@@ -65,5 +65,5 @@
       <visual>
         <geometry>
-          <mesh scale="0.001 0.001 0.001" filename="package://${package_name}/meshes/dragon_claw_claw_${digit}.stl"/>
+          <mesh scale="0.001 0.001 0.001" filename="package://${package_name}/openscad/stl/dragon_claw_claw_${digit}.stl"/>
         </geometry>
         <origin xyz="0 0 0" rpy="0 0 0"/>
